File: electrical/rotator_shield/rotator.sch (EAGLE design)
At the start: 10 parts, among them U1 OPTOISOLATOR

Commit message: Updated control pins
Connections:
- net GPIO18 renamed GPIO22
- removed net GPIO4: U1.A1
- new net GPIO23: B1.STEP
- net GPIO17: now also U1.A1; no longer B1.STEP
Changed lines of the file:
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@@
 <?xml version="1.0" encoding="utf-8"?>
 <!DOCTYPE eagle SYSTEM "eagle.dtd">
-<eagle version="8.6.0">
+<eagle version="9.1.3">
 <drawing>
 <settings>
@@
 <setting verticaltext="up"/>
 </settings>
-<grid distance="0.1" unitdist="inch" unit="inch" style="lines" multiple="1" display="yes" altdistance="0.01" altunitdist="inch" altunit="inch"/>
+<grid distance="0.1" unitdist="inch" unit="inch" style="lines" multiple="1" display="no" altdistance="0.01" altunitdist="inch" altunit="inch"/>
 <layers>
 <layer number="1" name="Top" color="4" fill="1" visible="no" active="no"/>
@@
 </segment>
 </net>
-<net name="GPIO4" class="0">
-<segment>
-<pinref part="U1" gate="G$1" pin="A1"/>
-<label x="68.58" y="96.52" size="1.778" layer="95"/>
-<wire x1="68.58" y1="96.52" x2="73.66" y2="96.52" width="0.1524" layer="91"/>
-</segment>
-</net>
 <net name="VSS" class="0">
 <segment>
@@
 <net name="GPIO17" class="0">
 <segment>
+<pinref part="U1" gate="G$1" pin="A1"/>
+<label x="68.58" y="96.52" size="1.778" layer="95"/>
+<wire x1="68.58" y1="96.52" x2="73.66" y2="96.52" width="0.1524" layer="91"/>
+</segment>
+</net>
+<net name="GPIO22" class="0">
+<segment>
+<pinref part="B1" gate="G$1" pin="DIR"/>
+<wire x1="38.1" y1="33.02" x2="25.4" y2="33.02" width="0.1524" layer="91"/>
+<label x="25.4" y="33.02" size="1.778" layer="95"/>
+</segment>
+</net>
+<net name="N$3" class="0">
+<segment>
+<pinref part="LED1" gate="G$1" pin="C"/>
+<pinref part="R1" gate="G$1" pin="2"/>
+<wire x1="55.88" y1="96.52" x2="55.88" y2="93.98" width="0.1524" layer="91"/>
+</segment>
+</net>
+<net name="N$7" class="0">
+<segment>
+<pinref part="U1" gate="G$1" pin="C1"/>
+<pinref part="R2" gate="G$1" pin="2"/>
+<wire x1="73.66" y1="93.98" x2="68.58" y2="93.98" width="0.1524" layer="91"/>
+</segment>
+</net>
+<net name="N$8" class="0">
+<segment>
+<pinref part="X1" gate="-1" pin="KL"/>
+<pinref part="S1" gate="1" pin="P"/>
+</segment>
+</net>
+<net name="GPIO23" class="0">
+<segment>
 <pinref part="B1" gate="G$1" pin="STEP"/>
 <wire x1="38.1" y1="35.56" x2="25.4" y2="35.56" width="0.1524" layer="91"/>
@@
 </segment>
 </net>
-<net name="GPIO18" class="0">
-<segment>
-<pinref part="B1" gate="G$1" pin="DIR"/>
-<wire x1="38.1" y1="33.02" x2="25.4" y2="33.02" width="0.1524" layer="91"/>
-<label x="25.4" y="33.02" size="1.778" layer="95"/>
-</segment>
-</net>
-<net name="N$3" class="0">
-<segment>
-<pinref part="LED1" gate="G$1" pin="C"/>
-<pinref part="R1" gate="G$1" pin="2"/>
-<wire x1="55.88" y1="96.52" x2="55.88" y2="93.98" width="0.1524" layer="91"/>
-</segment>
-</net>
-<net name="N$7" class="0">
-<segment>
-<pinref part="U1" gate="G$1" pin="C1"/>
-<pinref part="R2" gate="G$1" pin="2"/>
-<wire x1="73.66" y1="93.98" x2="68.58" y2="93.98" width="0.1524" layer="91"/>
-</segment>
-</net>
-<net name="N$8" class="0">
-<segment>
-<pinref part="X1" gate="-1" pin="KL"/>
-<pinref part="S1" gate="1" pin="P"/>
-</segment>
-</net>

Commit message: Added pull-down resistor to servo signal pin
Parts:
- added R3: 100, SparkFun-Resistors:68OHM-0603-1/10W-1%
- U1: value OPTOISOLATOR -> DUAL-OPTOISOLATOR_SOIC8
Connections:
- net GND: now also R3.1
- net N$1: now also R3.2
Changed lines of the file:
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@@
 </classes>
 <parts>
-<part name="U1" library="SparkFun-DiscreteSemi" deviceset="DUAL-OPTOISOLATOR" device="_SOIC8" value="OPTOISOLATOR"/>
+<part name="U1" library="SparkFun-DiscreteSemi" deviceset="DUAL-OPTOISOLATOR" device="_SOIC8" value=""/>
 <part name="SERVO" library="con-lstb" library_urn="urn:adsk.eagle:library:162" deviceset="MA03-1" device="" package3d_urn="urn:adsk.eagle:package:8339/1"/>
 <part name="P+1" library="supply1" library_urn="urn:adsk.eagle:library:371" deviceset="VCC" device=""/>
@@
 <part name="R2" library="SparkFun-Resistors" deviceset="68OHM" device="-0603-1/10W-1%" value="50"/>
 <part name="S1" library="SparkFun-Switches" deviceset="SWITCH-SPDT" device="-PTH-11.6X4.0MM"/>
+<part name="R3" library="SparkFun-Resistors" deviceset="68OHM" device="-0603-1/10W-1%" value="100"/>
 </parts>
 <sheets>
@@
 <instance part="R2" gate="G$1" x="68.58" y="88.9" rot="R90"/>
 <instance part="S1" gate="1" x="35.56" y="93.98"/>
+<instance part="R3" gate="G$1" x="96.52" y="86.36" rot="R180"/>
 </instances>
 <busses>
@@
 <wire x1="91.44" y1="106.68" x2="104.14" y2="106.68" width="0.1524" layer="91"/>
 <pinref part="PWR_GND" gate="1" pin="GND"/>
-<wire x1="104.14" y1="106.68" x2="104.14" y2="83.82" width="0.1524" layer="91"/>
+<wire x1="104.14" y1="106.68" x2="104.14" y2="86.36" width="0.1524" layer="91"/>
+<pinref part="R3" gate="G$1" pin="1"/>
+<wire x1="104.14" y1="86.36" x2="104.14" y2="83.82" width="0.1524" layer="91"/>
+<wire x1="101.6" y1="86.36" x2="104.14" y2="86.36" width="0.1524" layer="91"/>
+<junction x="104.14" y="86.36"/>
 </segment>
 </net>
@@
 <pinref part="U1" gate="G$1" pin="EM1"/>
 <pinref part="SERVO" gate="G$1" pin="1"/>
-<wire x1="86.36" y1="93.98" x2="91.44" y2="93.98" width="0.1524" layer="91"/>
+<wire x1="86.36" y1="93.98" x2="88.9" y2="93.98" width="0.1524" layer="91"/>
+<pinref part="R3" gate="G$1" pin="2"/>
+<wire x1="88.9" y1="93.98" x2="91.44" y2="93.98" width="0.1524" layer="91"/>
+<wire x1="91.44" y1="86.36" x2="88.9" y2="86.36" width="0.1524" layer="91"/>
+<wire x1="88.9" y1="86.36" x2="88.9" y2="93.98" width="0.1524" layer="91"/>
+<junction x="88.9" y="93.98"/>
 </segment>
 </net>
